File: pcb/RP2040_for_keebs.kicad_sch (KiCad schematic)
At the start: 31 parts, among them X1 S4T12000ZYFAC

Commit message: Add leds to schematic
Other:
- title: RP2040 for Keebs -> RP2040 Minimal Design for Keebs

Commit message: Update kicad schematics
Parts:
- U2: renamed from U1; footprint simplyKeeb:SOIC-8_L5.3-W5.3-P1.27-LS8.0-BL -> SOIC-8_L5.3-W5.3-P1.27-LS8.0-BL; LCSC Part (none) -> C82317
- U3: renamed from U2; footprint simplyKeeb:SOT-223-3_L6.5-W3.4-P2.30-LS7.0-BR -> SOT-223-3_L6.5-W3.4-P2.30-LS7.0-BR
- U4: renamed from U3; LCSC Part (none) -> C2040
- USB3: renamed from USB1; footprint simplyKeeb:USB-C-SMD_TYPE-C-31-M-31 -> USB-C-SMD_TYPE-C-31-M-31; LCSC Part (none) -> C2760486
- X1: footprint simplyKeeb:CRYSTAL-SMD_L7.4-W4.0-LS8.0 -> CRYSTAL-SMD_L7.4-W4.0-LS8.0; LCSC Part (none) -> C2149004
- renumbered C9 to C10, C10 to C11, C11 to C12, C12 to C13, C13 to C14, C14 to C15, C15 to C16, C16 to C17, C17 to C18, C1 to C3, C3 to C4, C4 to C5, C5 to C6, C6 to C7, C7 to C8, C8 to C9, R7 to R10, R1 to R4, R2 to R5, R3 to R6, R4 to R7, R5 to R8, R6 to R9, SW1 to SW61, SW2 to SW62
