File: pcb/Six-SK6812Mini-E.kicad_sch (KiCad schematic)
At the start: 12 parts

Commit message: Update kicad schematics
Other:
- moved on the sheet: C50, C51, C52, D69, D70

Commit message: Finalize schematic and start pcb led layout
Parts:
- renumbered C49 to C67, C50 to C68, C51 to C69, C52 to C70, C53 to C71, C54 to C72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
