File: pcb/simplyKeeb-60K.kicad_sch (KiCad schematic)
At the start: 127 parts, among them SW10 SW_Push, SW11 SW_Push, SW12 SW_Push, SW13 SW_Push, SW14 SW_Push, SW15 SW_Push, SW16 SW_Push, SW17 SW_Push, SW18 SW_Push, SW19 SW_Push, SW20 SW_Push, SW21 SW_Push, SW22 SW_Push, SW23 SW_Push, SW24 SW_Push, SW25 SW_Push, SW26 SW_Push, SW27 SW_Push, SW28 SW_Push, SW29 SW_Push, SW3 SW_Push, SW30 SW_Push, SW31 SW_Push, SW32 SW_Push, SW33 SW_Push, SW34 SW_Push, SW35 SW_Push, SW36 SW_Push, SW37 SW_Push, SW38 SW_Push, SW39 SW_Push, SW4 SW_Push, SW40 SW_Push, SW41 SW_Push, SW42 SW_Push, SW43 SW_Push, SW44 SW_Push, SW45 SW_Push, SW46 SW_Push, SW47 SW_Push, SW48 SW_Push, SW49 SW_Push, SW5 SW_Push, SW50 SW_Push, SW51 SW_Push, SW52 SW_Push, SW53 SW_Push, SW54 SW_Push, SW55 SW_Push, SW56 SW_Push, SW57 SW_Push, SW58 SW_Push, SW59 SW_Push, SW6 SW_Push, SW60 SW_Push, SW61 SW_Push, SW62 SW_Push, SW7 SW_Push, SW8 SW_Push, SW9 SW_Push, U10 PCA9555PW (IO Expander)

Commit message: Add leds to schematic
Connections:
- net I2C_SCL_L: no longer USB2.B6 (DP2)
- net I2C_SCL_R: no longer USB3.B6 (DP2)
- net I2C_SDA_L: no longer USB2.B7 (DN2)
- net I2C_SDA_R: no longer USB3.B7 (DN2)
- new net RGB_END_L: USB2.B6 (DP2)
- new net RGB_START_R: USB3.B6 (DP2)
- no-connect marks 30 -> 32
Other:
- added sheet Six SK6812Mini-E (Six-SK6812Mini-E.kicad_sch)
- added sheet Six SK6812Mini-E1 (Six-SK6812Mini-E.kicad_sch)
- added sheet Six SK6812Mini-E10 (Six-SK6812Mini-E.kicad_sch)
- added sheet Six SK6812Mini-E11 (Six-SK6812Mini-E.kicad_sch)
- added sheet Six SK6812Mini-E12 (Six-SK6812Mini-E.kicad_sch)
- added sheet Six SK6812Mini-E13 (Six-SK6812Mini-E.kicad_sch)
- added sheet Six SK6812Mini-E14 (Six-SK6812Mini-E.kicad_sch)
- added sheet Six SK6812Mini-E15 (Six-SK6812Mini-E.kicad_sch)
- added sheet Six SK6812Mini-E16 (Six-SK6812Mini-E.kicad_sch)
- added sheet Six SK6812Mini-E17 (Six-SK6812Mini-E.kicad_sch)
- added sheet Six SK6812Mini-E2 (Six-SK6812Mini-E.kicad_sch)
- added sheet Six SK6812Mini-E3 (Six-SK6812Mini-E.kicad_sch)
- added sheet Six SK6812Mini-E4 (Six-SK6812Mini-E.kicad_sch)
- added sheet Six SK6812Mini-E5 (Six-SK6812Mini-E.kicad_sch)
- added sheet Six SK6812Mini-E6 (Six-SK6812Mini-E.kicad_sch)
- added sheet Six SK6812Mini-E7 (Six-SK6812Mini-E.kicad_sch)
- added sheet Six SK6812Mini-E8 (Six-SK6812Mini-E.kicad_sch)
- added sheet Six SK6812Mini-E9 (Six-SK6812Mini-E.kicad_sch)
- note added: "Backlight"
- note added: "End of the right half go into one of the split USB C connection wires. And starts again on the keys of the right half. The order is L-Backlight, L-PerKey, R-PerKey, R-Backlight."
- note added: "Per Key LEDs"
- title: simplyKeeb-T36 -> simplyKeeb-S60
- moved on the sheet: C18, D10, D100, D106, D107, D108, D109, D110, D116, D117, D118, D119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

Commit message: Update kicad schematics
Parts:
- U1: renamed from U10; footprint simplyKeeb:TSSOP-24_L7.8-W4.4-P0.65-LS6.4-BL -> TSSOP-24_L7.8-W4.4-P0.65-LS6.4-BL; LCSC Part (none) -> C128392
- USB1: renamed from USB3; footprint simplyKeeb:USB-C-SMD_TYPE-C-31-M-31 -> USB-C-SMD_TYPE-C-31-M-31; LCSC Part (none) -> C2760486
- USB2: footprint simplyKeeb:USB-C-SMD_TYPE-C-31-M-31 -> USB-C-SMD_TYPE-C-31-M-31; LCSC Part (none) -> C2760486
- renumbered C18 to C1, D6 to D1, D20 to D10, D61 to D11, D62 to D12, D63 to D13, D64 to D14, D65 to D15, D26 to D16, D27 to D17, D28 to D18, D29 to D19, D7 to D2, D30 to D20, D71 to D21, D72 to D22, D73 to D23, D74 to D24, D75 to D25, D36 to D26, D37 to D27, D38 to D28, D39 to D29, D8 to D3, D40 to D30, D86 to D31, D87 to D32, D88 to D33, D89 to D34, D90 to D35, D46 to D36, D47 to D37, D48 to D38, D49 to D39, D9 to D4, D50 to D40, D96 to D41, D97 to D42, D98 to D43, D99 to D44, D100 to D45, D56 to D46, D57 to D47, D58 to D48, D59 to D49, D10 to D5, D60 to D50, D106 to D51, D107 to D52, D108 to D53, D109 to D54, D110 to D55, D116 to D56, D117 to D57, D118 to D58, D119 to D59, D16 to D6, D120 to D60, D17 to D7, D18 to D8, D19 to D9, R8 to R1, R9 to R2, R10 to R3, SW3 to SW1, SW12 to SW10, SW33 to SW11, SW34 to SW12, SW35 to SW13, SW36 to SW14, SW37 to SW15, SW13 to SW16, SW14 to SW17, SW15 to SW18, SW16 to SW19, SW4 to SW2, SW17 to SW20, SW38 to SW21, SW39 to SW22, SW40 to SW23, SW41 to SW24, SW42 to SW25, SW18 to SW26, SW19 to SW27, SW20 to SW28, SW21 to SW29, SW5 to SW3, SW22 to SW30, SW43 to SW31, SW44 to SW32, SW45 to SW33, SW46 to SW34, SW47 to SW35, SW23 to SW36, SW24 to SW37, SW25 to SW38, SW26 to SW39, SW6 to SW4, SW27 to SW40, SW48 to SW41, SW49 to SW42, SW50 to SW43, SW51 to SW44, SW52 to SW45, SW28 to SW46, SW29 to SW47, SW30 to SW48, SW31 to SW49, SW7 to SW5, SW32 to SW50, SW53 to SW51, SW54 to SW52, SW55 to SW53, SW56 to SW54, SW57 to SW55, SW58 to SW56, SW59 to SW57, SW60 to SW58, SW61 to SW59, SW8 to SW6, SW62 to SW60, SW9 to SW7, SW10 to SW8, SW11 to SW9
Other:
- sheet Six SK6812Mini-E10 renamed Four SK6812Mini-E10
- sheet Six SK6812Mini-E16 renamed Four SK6812Mini-E16
- sheet Six SK6812Mini-E17 renamed Four SK6812Mini-E17
- sheet Six SK6812Mini-E5 renamed Four SK6812Mini-E5
- sheet Six SK6812Mini-E6 renamed Four SK6812Mini-E6
- sheet Six SK6812Mini-E7 renamed Four SK6812Mini-E7
- sheet Six SK6812Mini-E8 renamed Four SK6812Mini-E8
- sheet Six SK6812Mini-E9 renamed Four SK6812Mini-E9
- sheet Four SK6812Mini-E10: file Six-SK6812Mini-E.kicad_sch -> Four-SK6812Mini-E.kicad_sch
- sheet Four SK6812Mini-E16: file Six-SK6812Mini-E.kicad_sch -> Four-SK6812Mini-E.kicad_sch
- sheet Four SK6812Mini-E17: file Six-SK6812Mini-E.kicad_sch -> Four-SK6812Mini-E.kicad_sch
- sheet Four SK6812Mini-E5: file Six-SK6812Mini-E.kicad_sch -> Four-SK6812Mini-E.kicad_sch
- sheet Four SK6812Mini-E6: file Six-SK6812Mini-E.kicad_sch -> Four-SK6812Mini-E.kicad_sch
- sheet Four SK6812Mini-E7: file Six-SK6812Mini-E.kicad_sch -> Four-SK6812Mini-E.kicad_sch
- sheet Four SK6812Mini-E8: file Six-SK6812Mini-E.kicad_sch -> Four-SK6812Mini-E.kicad_sch
- sheet Four SK6812Mini-E9: file Six-SK6812Mini-E.kicad_sch -> Four-SK6812Mini-E.kicad_sch
- moved on the sheet: C1, D1, D10, D11, D12, D13, D14, D15, D16, D17, D18, D19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

Commit message: Finalize schematic and start pcb led layout
Other:
- sheet Four SK6812Mini-E16 renamed Six SK6812Mini-E16
- sheet Four SK6812Mini-E17 renamed Six SK6812Mini-E17
- sheet Four SK6812Mini-E5 renamed Six SK6812Mini-E5
- sheet Four SK6812Mini-E6 renamed Six SK6812Mini-E6
- sheet Four SK6812Mini-E7 renamed Six SK6812Mini-E7
- sheet Four SK6812Mini-E9 renamed Six SK6812Mini-E9
- sheet Six SK6812Mini-E16: file Four-SK6812Mini-E.kicad_sch -> Six-SK6812Mini-E.kicad_sch
- sheet Six SK6812Mini-E17: file Four-SK6812Mini-E.kicad_sch -> Six-SK6812Mini-E.kicad_sch
- sheet Six SK6812Mini-E5: file Four-SK6812Mini-E.kicad_sch -> Six-SK6812Mini-E.kicad_sch
- sheet Six SK6812Mini-E6: file Four-SK6812Mini-E.kicad_sch -> Six-SK6812Mini-E.kicad_sch
- sheet Six SK6812Mini-E7: file Four-SK6812Mini-E.kicad_sch -> Six-SK6812Mini-E.kicad_sch
- sheet Six SK6812Mini-E9: file Four-SK6812Mini-E.kicad_sch -> Six-SK6812Mini-E.kicad_sch
Changed lines of the file:
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@@
     (stroke (width 0.1524) (type solid))
     (fill (color 0 0 0 0.0000))
-    (property "Sheetname" "Four SK6812Mini-E6" (at 401.32 126.2884 0)
-      (effects (font (size 1.27 1.27)) (justify left bottom))
-    )
-    (property "Sheetfile" "Four-SK6812Mini-E.kicad_sch" (at 401.32 135.9666 0)
+    (property "Sheetname" "Six SK6812Mini-E6" (at 401.32 126.2884 0)
+      (effects (font (size 1.27 1.27)) (justify left bottom))
+    )
+    (property "Sheetfile" "Six-SK6812Mini-E.kicad_sch" (at 401.32 135.9666 0)
       (effects (font (size 1.27 1.27)) (justify left top))
     )
@@
     (stroke (width 0.1524) (type solid))
     (fill (color 0 0 0 0.0000))
-    (property "Sheetname" "Four SK6812Mini-E16" (at 481.33 268.5284 0)
-      (effects (font (size 1.27 1.27)) (justify left bottom))
-    )
-    (property "Sheetfile" "Four-SK6812Mini-E.kicad_sch" (at 481.33 278.2066 0)
+    (property "Sheetname" "Six SK6812Mini-E16" (at 481.33 268.5284 0)
+      (effects (font (size 1.27 1.27)) (justify left bottom))
+    )
+    (property "Sheetfile" "Six-SK6812Mini-E.kicad_sch" (at 481.33 278.2066 0)
       (effects (font (size 1.27 1.27)) (justify left top))
     )
@@
     (stroke (width 0.1524) (type solid))
     (fill (color 0 0 0 0.0000))
-    (property "Sheetname" "Four SK6812Mini-E5" (at 401.32 111.0484 0)
-      (effects (font (size 1.27 1.27)) (justify left bottom))
-    )
-    (property "Sheetfile" "Four-SK6812Mini-E.kicad_sch" (at 401.32 120.7266 0)
+    (property "Sheetname" "Six SK6812Mini-E5" (at 401.32 111.0484 0)
+      (effects (font (size 1.27 1.27)) (justify left bottom))
+    )
+    (property "Sheetfile" "Six-SK6812Mini-E.kicad_sch" (at 401.32 120.7266 0)
       (effects (font (size 1.27 1.27)) (justify left top))
     )
@@
     (stroke (width 0.1524) (type solid))
     (fill (color 0 0 0 0.0000))
-    (property "Sheetname" "Four SK6812Mini-E7" (at 401.32 144.0684 0)
-      (effects (font (size 1.27 1.27)) (justify left bottom))
-    )
-    (property "Sheetfile" "Four-SK6812Mini-E.kicad_sch" (at 401.32 153.7466 0)
+    (property "Sheetname" "Six SK6812Mini-E7" (at 401.32 144.0684 0)
+      (effects (font (size 1.27 1.27)) (justify left bottom))
+    )
+    (property "Sheetfile" "Six-SK6812Mini-E.kicad_sch" (at 401.32 153.7466 0)
       (effects (font (size 1.27 1.27)) (justify left top))
     )
@@
     (stroke (width 0.1524) (type solid))
     (fill (color 0 0 0 0.0000))
-    (property "Sheetname" "Four SK6812Mini-E17" (at 481.33 283.7684 0)
-      (effects (font (size 1.27 1.27)) (justify left bottom))
-    )
-    (property "Sheetfile" "Four-SK6812Mini-E.kicad_sch" (at 481.33 293.4466 0)
+    (property "Sheetname" "Six SK6812Mini-E17" (at 481.33 283.7684 0)
+      (effects (font (size 1.27 1.27)) (justify left bottom))
+    )
+    (property "Sheetfile" "Six-SK6812Mini-E.kicad_sch" (at 481.33 293.4466 0)
       (effects (font (size 1.27 1.27)) (justify left top))
     )
@@
     (stroke (width 0.1524) (type solid))
     (fill (color 0 0 0 0.0000))
-    (property "Sheetname" "Four SK6812Mini-E9" (at 481.33 301.5484 0)
-      (effects (font (size 1.27 1.27)) (justify left bottom))
-    )
-    (property "Sheetfile" "Four-SK6812Mini-E.kicad_sch" (at 481.33 311.2266 0)
-      (effects (font (size 1.27 1.27)) (justify left top))
-    )
+    (property "Sheetname" "Six SK6812Mini-E9" (at 481.33 301.5484 0)
+      (effects (font (size 1.27 1.27)) (justify left bottom))
+    )
+    (property "Sheetfile" "Six-SK6812Mini-E.kicad_sch" (at 481.33 311.2266 0)
+      (effects (font (size 1.27 1.27)) (justify left top))
+    )
