File: splitchoc/pcb/Five-SK6812Mini-E.kicad_sch (KiCad schematic)
At the start: 8 parts

Commit message: Version update and add s60c
Parts:
- added C78: C, Capacitor_SMD:C_0402_1005Metric, symbol Device:C
- added D115: SK6812MINI-E, simplyKeeb:Choc_SK6812MINI-E, symbol simplyKeeb:SK6812MINI-E
- D105, D111, D112, D115: footprint simplyKeeb:MX_SK6812MINI-E -> simplyKeeb:Choc_SK6812MINI-E
Connections:
- net DOUT: now also D115.2 (DOUT); no longer D115.2 (DOUT)
- net GND: now also C78.2, D115.3 (GND)
- net VBUS: now also C78.1, D115.1 (VDD)
- new net: D115.2 (DOUT), D115.4 (DIN)
