File: splitchoc/pcb/RP2040_for_keebs.kicad_sch (KiCad schematic)
At the start: 31 parts, among them X1 S4T12000ZYFAC

Commit message: Version update and add s60c
Parts:
- U2: footprint SOIC-8_L5.3-W5.3-P1.27-LS8.0-BL -> simplyKeeb:SOIC-8_L5.3-W5.3-P1.27-LS8.0-BL
- U3: footprint SOT-223-3_L6.5-W3.4-P2.30-LS7.0-BR -> simplyKeeb:SOT-223-3_L6.5-W3.4-P2.30-LS7.0-BR
- USB3: footprint USB-C-SMD_TYPE-C-31-M-31 -> simplyKeeb:USB-C-SMD_TYPE-C-31-M-31
- X1: footprint CRYSTAL-SMD_L7.4-W4.0-LS8.0 -> simplyKeeb:CRYSTAL-SMD_L7.4-W4.0-LS8.0
