File: splitchoc/pcb/Six-SK6812Mini-E.kicad_sch (KiCad schematic)
At the start: 12 parts

Commit message: Version update and add s60c
Parts:
- D101, D102, D103, D104, D94, D95: footprint simplyKeeb:MX_SK6812MINI-E -> simplyKeeb:Choc_SK6812MINI-E
Connections:
- net GND: now also C69.1; no longer C69.2
- net VBUS: now also C69.2; no longer C69.1
Changed lines of the file:
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@@
     (effects (font (size 1.27 1.27)) (justify left))
   )
-  (symbol (lib_id "Device:C") (at 120.65 78.74 0) (mirror y) (unit 1)
-    (in_bom yes) (on_board yes) (dnp no) (fields_autoplaced)
-    (property "Reference" "C69" (at 117.729 77.9053 0)
-      (effects (font (size 1.27 1.27)) (justify left))
-    )
-    (property "Value" "C" (at 117.729 80.4422 0)
-      (effects (font (size 1.27 1.27)) (justify left))
-    )
-    (property "Footprint" "Capacitor_SMD:C_0402_1005Metric" (at 119.6848 82.55 0)
+  (symbol (lib_id "Device:C") (at 120.65 78.74 0) (mirror x) (unit 1)
+    (in_bom yes) (on_board yes) (dnp no) (fields_autoplaced)
+    (property "Reference" "C69" (at 116.84 78.105 0)
+      (effects (font (size 1.27 1.27)) (justify right))
+    )
+    (property "Value" "C" (at 116.84 80.645 0)
+      (effects (font (size 1.27 1.27)) (justify right))
+    )
+    (property "Footprint" "Capacitor_SMD:C_0402_1005Metric" (at 121.6152 74.93 0)
       (effects (font (size 1.27 1.27)) hide)
     )
@@
     (pin "2")
     (instances
-      (project "simplyKeeb-60K"
+      (project "simplyKeeb-S60c"
         (path "/3ef7093d-56c4-42ac-a29c-e335ba172a8b/de743d67-c1f2-4b03-b35a-3f0fd7f4a0ff"
           (reference "C69") (unit 1)
@@
     (pin "1")
     (instances
-      (project "simplyKeeb-60K"
+      (project "simplyKeeb-S60c"
         (path "/3ef7093d-56c4-42ac-a29c-e335ba172a8b/de743d67-c1f2-4b03-b35a-3f0fd7f4a0ff"
           (reference "#PWR0178") (unit 1)
@@
       (effects (font (size 1.27 1.27)) (justify left bottom))
     )
-    (property "Footprint" "simplyKeeb:MX_SK6812MINI-E" (at 190.5 87.63 0)
+    (property "Footprint" "simplyKeeb:Choc_SK6812MINI-E" (at 190.5 87.63 0)
       (effects (font (size 1.27 1.27)) hide)
     )
@@
     (pin "4")
     (instances
-      (project "simplyKeeb-60K"
+      (project "simplyKeeb-S60c"
         (path "/3ef7093d-56c4-42ac-a29c-e335ba172a8b/de743d67-c1f2-4b03-b35a-3f0fd7f4a0ff"
           (reference "D103") (unit 1)
@@
     (pin "1")
     (instances
-      (project "simplyKeeb-60K"
+      (project "simplyKeeb-S60c"
         (path "/3ef7093d-56c4-42ac-a29c-e335ba172a8b/de743d67-c1f2-4b03-b35a-3f0fd7f4a0ff"
           (reference "#PWR0185") (unit 1)
@@
     (pin "1")
     (instances
-      (project "simplyKeeb-60K"
+      (project "simplyKeeb-S60c"
         (path "/3ef7093d-56c4-42ac-a29c-e335ba172a8b/de743d67-c1f2-4b03-b35a-3f0fd7f4a0ff"
           (reference "#PWR0179") (unit 1)
@@
       (effects (font (size 1.27 1.27)) (justify left bottom))
     )
-    (property "Footprint" "simplyKeeb:MX_SK6812MINI-E" (at 163.83 87.63 0)
+    (property "Footprint" "simplyKeeb:Choc_SK6812MINI-E" (at 163.83 87.63 0)
       (effects (font (size 1.27 1.27)) hide)
     )
@@
     (pin "4")
     (instances
-      (project "simplyKeeb-60K"
+      (project "simplyKeeb-S60c"
         (path "/3ef7093d-56c4-42ac-a29c-e335ba172a8b/de743d67-c1f2-4b03-b35a-3f0fd7f4a0ff"
           (reference "D102") (unit 1)
@@
     (pin "2")
     (instances
-      (project "simplyKeeb-60K"
+      (project "simplyKeeb-S60c"
         (path "/3ef7093d-56c4-42ac-a29c-e335ba172a8b/de743d67-c1f2-4b03-b35a-3f0fd7f4a0ff"
           (reference "C71") (unit 1)
@@
     (pin "1")
     (instances
-      (project "simplyKeeb-60K"
+      (project "simplyKeeb-S60c"
         (path "/3ef7093d-56c4-42ac-a29c-e335ba172a8b/de743d67-c1f2-4b03-b35a-3f0fd7f4a0ff"
           (reference "#PWR0190") (unit 1)
@@
     (pin "1")
     (instances
-      (project "simplyKeeb-60K"
+      (project "simplyKeeb-S60c"
         (path "/3ef7093d-56c4-42ac-a29c-e335ba172a8b/de743d67-c1f2-4b03-b35a-3f0fd7f4a0ff"
           (reference "#PWR0180") (unit 1)
@@
     (pin "1")
     (instances
-      (project "simplyKeeb-60K"
+      (project "simplyKeeb-S60c"
         (path "/3ef7093d-56c4-42ac-a29c-e335ba172a8b/de743d67-c1f2-4b03-b35a-3f0fd7f4a0ff"
           (reference "#PWR0177") (unit 1)
@@
     (pin "1")
     (instances
-      (project "simplyKeeb-60K"
+      (project "simplyKeeb-S60c"
         (path "/3ef7093d-56c4-42ac-a29c-e335ba172a8b/de743d67-c1f2-4b03-b35a-3f0fd7f4a0ff"
           (reference "#PWR0187") (unit 1)
@@
       (effects (font (size 1.27 1.27)) (justify left bottom))
     )
-    (property "Footprint" "simplyKeeb:MX_SK6812MINI-E" (at 219.71 87.63 0)
+    (property "Footprint" "simplyKeeb:Choc_SK6812MINI-E" (at 219.71 87.63 0)
       (effects (font (size 1.27 1.27)) hide)
     )
@@
     (pin "4")
     (instances
-      (project "simplyKeeb-60K"
+      (project "simplyKeeb-S60c"
         (path "/3ef7093d-56c4-42ac-a29c-e335ba172a8b/de743d67-c1f2-4b03-b35a-3f0fd7f4a0ff"
           (reference "D104") (unit 1)
@@
     (pin "1")
     (instances
-      (project "simplyKeeb-60K"
+      (project "simplyKeeb-S60c"
         (path "/3ef7093d-56c4-42ac-a29c-e335ba172a8b/de743d67-c1f2-4b03-b35a-3f0fd7f4a0ff"
           (reference "#PWR0175") (unit 1)
@@
     (pin "1")
     (instances
-      (project "simplyKeeb-60K"
+      (project "simplyKeeb-S60c"
         (path "/3ef7093d-56c4-42ac-a29c-e335ba172a8b/de743d67-c1f2-4b03-b35a-3f0fd7f4a0ff"
           (reference "#PWR0181") (unit 1)
@@
     (pin "1")
     (instances
-      (project "simplyKeeb-60K"
+      (project "simplyKeeb-S60c"
         (path "/3ef7093d-56c4-42ac-a29c-e335ba172a8b/de743d67-c1f2-4b03-b35a-3f0fd7f4a0ff"
           (reference "#PWR0189") (unit 1)
@@
     (pin "2")
     (instances
-      (project "simplyKeeb-60K"
+      (project "simplyKeeb-S60c"
         (path "/3ef7093d-56c4-42ac-a29c-e335ba172a8b/de743d67-c1f2-4b03-b35a-3f0fd7f4a0ff"
           (reference "C67") (unit 1)
@@
     (pin "2")
     (instances
-      (project "simplyKeeb-60K"
+      (project "simplyKeeb-S60c"
         (path "/3ef7093d-56c4-42ac-a29c-e335ba172a8b/de743d67-c1f2-4b03-b35a-3f0fd7f4a0ff"
           (reference "C70") (unit 1)
@@
     (pin "1")
     (instances
-      (project "simplyKeeb-60K"
+      (project "simplyKeeb-S60c"
         (path "/3ef7093d-56c4-42ac-a29c-e335ba172a8b/de743d67-c1f2-4b03-b35a-3f0fd7f4a0ff"
           (reference "#PWR0188") (unit 1)
@@
     (pin "2")
     (instances
-      (project "simplyKeeb-60K"
+      (project "simplyKeeb-S60c"
         (path "/3ef7093d-56c4-42ac-a29c-e335ba172a8b/de743d67-c1f2-4b03-b35a-3f0fd7f4a0ff"
           (reference "C68") (unit 1)
@@
     (pin "2")
     (instances
-      (project "simplyKeeb-60K"
+      (project "simplyKeeb-S60c"
         (path "/3ef7093d-56c4-42ac-a29c-e335ba172a8b/de743d67-c1f2-4b03-b35a-3f0fd7f4a0ff"
           (reference "C72") (unit 1)
@@
     (pin "1")
     (instances
-      (project "simplyKeeb-60K"
+      (project "simplyKeeb-S60c"
         (path "/3ef7093d-56c4-42ac-a29c-e335ba172a8b/de743d67-c1f2-4b03-b35a-3f0fd7f4a0ff"
           (reference "#PWR0176") (unit 1)
@@
     (pin "1")
     (instances
-      (project "simplyKeeb-60K"
+      (project "simplyKeeb-S60c"
         (path "/3ef7093d-56c4-42ac-a29c-e335ba172a8b/de743d67-c1f2-4b03-b35a-3f0fd7f4a0ff"
           (reference "#PWR0183") (unit 1)
@@
     (pin "1")
     (instances
-      (project "simplyKeeb-60K"
+      (project "simplyKeeb-S60c"
         (path "/3ef7093d-56c4-42ac-a29c-e335ba172a8b/de743d67-c1f2-4b03-b35a-3f0fd7f4a0ff"
           (reference "#PWR0192") (unit 1)
@@
     (pin "1")
     (instances
-      (project "simplyKeeb-60K"
+      (project "simplyKeeb-S60c"
         (path "/3ef7093d-56c4-42ac-a29c-e335ba172a8b/de743d67-c1f2-4b03-b35a-3f0fd7f4a0ff"
           (reference "#PWR0186") (unit 1)
@@
     (pin "1")
     (instances
-      (project "simplyKeeb-60K"
+      (project "simplyKeeb-S60c"
         (path "/3ef7093d-56c4-42ac-a29c-e335ba172a8b/de743d67-c1f2-4b03-b35a-3f0fd7f4a0ff"
           (reference "#PWR0182") (unit 1)
@@
     (pin "1")
     (instances
-      (project "simplyKeeb-60K"
+      (project "simplyKeeb-S60c"
         (path "/3ef7093d-56c4-42ac-a29c-e335ba172a8b/de743d67-c1f2-4b03-b35a-3f0fd7f4a0ff"
           (reference "#PWR0184") (unit 1)
@@
       (effects (font (size 1.27 1.27)) (justify left bottom))
     )
-    (property "Footprint" "simplyKeeb:MX_SK6812MINI-E" (at 105.41 87.63 0)
+    (property "Footprint" "simplyKeeb:Choc_SK6812MINI-E" (at 105.41 87.63 0)
       (effects (font (size 1.27 1.27)) hide)
     )
@@
     (pin "4")
     (instances
-      (project "simplyKeeb-60K"
+      (project "simplyKeeb-S60c"
         (path "/3ef7093d-56c4-42ac-a29c-e335ba172a8b/de743d67-c1f2-4b03-b35a-3f0fd7f4a0ff"
           (reference "D95") (unit 1)
@@
       (effects (font (size 1.27 1.27)) (justify left bottom))
     )
-    (property "Footprint" "simplyKeeb:MX_SK6812MINI-E" (at 134.62 87.63 0)
+    (property "Footprint" "simplyKeeb:Choc_SK6812MINI-E" (at 134.62 87.63 0)
       (effects (font (size 1.27 1.27)) hide)
     )
@@
     (pin "4")
     (instances
-      (project "simplyKeeb-60K"
+      (project "simplyKeeb-S60c"
         (path "/3ef7093d-56c4-42ac-a29c-e335ba172a8b/de743d67-c1f2-4b03-b35a-3f0fd7f4a0ff"
           (reference "D101") (unit 1)
@@
       (effects (font (size 1.27 1.27)) (justify left bottom))
     )
-    (property "Footprint" "simplyKeeb:MX_SK6812MINI-E" (at 76.2 87.63 0)
+    (property "Footprint" "simplyKeeb:Choc_SK6812MINI-E" (at 76.2 87.63 0)
       (effects (font (size 1.27 1.27)) hide)
     )
@@
     (pin "4")
     (instances
-      (project "simplyKeeb-60K"
+      (project "simplyKeeb-S60c"
         (path "/3ef7093d-56c4-42ac-a29c-e335ba172a8b/de743d67-c1f2-4b03-b35a-3f0fd7f4a0ff"
           (reference "D94") (unit 1)
@@
     (pin "1")
     (instances
-      (project "simplyKeeb-60K"
+      (project "simplyKeeb-S60c"
         (path "/3ef7093d-56c4-42ac-a29c-e335ba172a8b/de743d67-c1f2-4b03-b35a-3f0fd7f4a0ff"
           (reference "#PWR0191") (unit 1)
