File: splitchoc/pcb/simplyKeeb-S60c.kicad_sch (KiCad schematic)
At the start: 127 parts, among them SW1 SW_Push, SW10 SW_Push, SW11 SW_Push, SW12 SW_Push, SW13 SW_Push, SW14 SW_Push, SW15 SW_Push, SW16 SW_Push, SW17 SW_Push, SW18 SW_Push, SW19 SW_Push, SW2 SW_Push, SW20 SW_Push, SW21 SW_Push, SW22 SW_Push, SW23 SW_Push, SW24 SW_Push, SW25 SW_Push, SW26 SW_Push, SW27 SW_Push, SW28 SW_Push, SW29 SW_Push, SW3 SW_Push, SW30 SW_Push, SW31 SW_Push, SW32 SW_Push, SW33 SW_Push, SW34 SW_Push, SW35 SW_Push, SW36 SW_Push, SW37 SW_Push, SW38 SW_Push, SW39 SW_Push, SW4 SW_Push, SW40 SW_Push, SW41 SW_Push, SW42 SW_Push, SW43 SW_Push, SW44 SW_Push, SW45 SW_Push, SW46 SW_Push, SW47 SW_Push, SW48 SW_Push, SW49 SW_Push, SW5 SW_Push, SW50 SW_Push, SW51 SW_Push, SW52 SW_Push, SW53 SW_Push, SW54 SW_Push, SW55 SW_Push, SW56 SW_Push, SW57 SW_Push, SW58 SW_Push, SW59 SW_Push, SW6 SW_Push, SW60 SW_Push, SW7 SW_Push, SW8 SW_Push, SW9 SW_Push, U1 PCA9555PW (IO Expander)

Commit message: Version update and add s60c
Parts:
- SW1, SW10, SW11, SW12, SW13, SW14, SW16, SW17, SW18, SW19, SW2, SW20, SW21, SW22, SW23, SW24, SW26, SW27, SW28, SW29, SW3, SW30, SW31, SW32, SW33, SW34, SW35, SW36, SW37, SW38, SW39, SW4, SW41, SW42, SW43, SW44, SW45, SW46, SW47, SW48, SW49, SW5, SW51, SW52, SW53, SW54, SW55, SW56, SW57, SW58, SW59, SW6, SW60, SW7, SW8, SW9: footprint simplyKeeb:MXOnly-1U-Hotswap -> simplyKeeb:Choc-1U-Hotswap
- SW15, SW50: footprint simplyKeeb:MXOnly-2U-Hotswap-Vertical -> simplyKeeb:Choc-2U-Hotswap-Vertical
- SW25, SW40: footprint simplyKeeb:MXOnly-1.5U-Hotswap-Vertical -> simplyKeeb:Choc-1.5U-Hotswap-Vertical
- U1: footprint TSSOP-24_L7.8-W4.4-P0.65-LS6.4-BL -> simplyKeeb:TSSOP-24_L7.8-W4.4-P0.65-LS6.4-BL
- USB1, USB2: footprint USB-C-SMD_TYPE-C-31-M-31 -> simplyKeeb:USB-C-SMD_TYPE-C-31-M-31
Other:
- sheet Four SK6812Mini-E10 renamed Backlight R4
- sheet Four SK6812Mini-E8 renamed Backlight L4
- sheet Six SK6812Mini-E renamed LEDs Row L1
- sheet Six SK6812Mini-E1 renamed LEDs Row L2
- sheet Six SK6812Mini-E11 renamed LEDs Row R5
- sheet Six SK6812Mini-E12 renamed LEDs Row R4
- sheet Six SK6812Mini-E13 renamed LEDs Row R3
- sheet Six SK6812Mini-E14 renamed LEDs Row R2
- sheet Six SK6812Mini-E15 renamed LEDs Row R1
- sheet Six SK6812Mini-E16 renamed Backlight R1
- sheet Six SK6812Mini-E17 renamed Backlight R2
- sheet Six SK6812Mini-E2 renamed LEDs Row L3
- sheet Six SK6812Mini-E3 renamed LEDs Row L4
- sheet Six SK6812Mini-E4 renamed LEDs Row L5
- sheet Six SK6812Mini-E5 renamed Backlight L1
- sheet Six SK6812Mini-E6 renamed Backlight L2
- sheet Six SK6812Mini-E7 renamed Backlight L3
- sheet Six SK6812Mini-E9 renamed Backlight R3
- sheet Backlight L4: file Four-SK6812Mini-E.kicad_sch -> Five-SK6812Mini-E.kicad_sch
- sheet Backlight R4: file Four-SK6812Mini-E.kicad_sch -> Five-SK6812Mini-E.kicad_sch
